Commit message: gazeno できない

File: wheel_description/urdf/wheel.xacro (robot description, xacro)
@@ -107,5 +107,5 @@
     <child link="right_wheel"/>
     <parent link="base_link"/>
-    <axis xyz="0 0 1" rpy="0 0 0"/>
+    <axis xyz="0 0 -1" rpy="0 0 0"/>
     <limit effort="10000" velocity="1000"/>
     <joint_properties damping="1.0" friction="1.0"/>
@@ -137,3 +137,22 @@
     <child link="hokuyo_link"/>
   </joint>
+  <gazebo>
+    <plugin name="differential_drive_controller" filename="libgazebo_ros_diff_drive.so">
+      <legacyMode>false</legacyMode>
+      <alwaysOn>true</alwaysOn>
+      <updateRate>20</updateRate>
+      <leftJoint>left_wheel_hinge</leftJoint>
+      <rightJoint>right_wheel_hinge</rightJoint>
+      <wheelSeparation>0.4</wheelSeparation>
+      <wheelDiameter>0.1</wheelDiameter>
+      <torque>20</torque>
+      <commandTopic>cmd_vel</commandTopic>
+      <odometryTopic>odom</odometryTopic>
+      <odometryFrame>odom</odometryFrame>
+      <robotBaseFrame>chassis</robotBaseFrame>
+    </plugin>
+  </gazebo>
+  <gazebo reference="chassis">
+      <material>Gazebo/Orange</material>
+    </gazebo>
 </robot>

Commit message: added base_imu_link robot_pose_ekf

File: wheel_description/urdf/wheel.xacro (robot description, xacro)
@@ -52,5 +52,5 @@
       <origin xyz="0 0 0" rpy="0 0 0"/>
       <geometry>
-        <cylinder radius="0.28" length="0.05"/>
+        <cylinder radius="0.2794" length="0.05"/>
       </geometry>
     </collision>
@@ -58,5 +58,5 @@
       <origin xyz="0 0 0" rpy="0 0 0"/>
       <geometry>
-        <cylinder radius="0.28" length="0.05"/>
+        <cylinder radius="0.2794" length="0.05"/>
       </geometry>
     </visual>
@@ -75,5 +75,5 @@
       <origin xyz="0 0 0" rpy="0 0 0"/>
       <geometry>
-        <cylinder radius="0.28" length="0.05"/>
+        <cylinder radius="0.2794" length="0.05"/>
       </geometry>
     </collision>
@@ -81,5 +81,5 @@
       <origin xyz="0 0 0" rpy="0 0 0"/>
       <geometry>
-        <cylinder radius="0.28" length="0.05"/>
+        <cylinder radius="0.2794" length="0.05"/>
       </geometry>
     </visual>
@@ -137,4 +137,23 @@
     <child link="hokuyo_link"/>
   </joint>
+ <link name="base_imu_link">
+    <collision>
+      <origin xyz="0 0 0" rpy="0 0 0"/>
+      <geometry>
+        <box size="0.1 0.1 0.1"/>
+      </geometry>
+    </collision>
+    <inertial>
+      <mass value="1e-5" />
+      <origin xyz="0 0 0" rpy="0 0 0"/>
+      <inertia ixx="1e-6" ixy="0" ixz="0" iyy="1e-6" iyz="0" izz="1e-6" />
+    </inertial>
+  </link>
+ <joint name="imu_joint" type="fixed">
+    <axis xyz="0 0 0" />
+    <origin xyz="0 0 0.75" rpy="0 0 0"/>
+    <parent link="base_link"/>
+    <child link="base_imu_link"/>
+  </joint>
   <gazebo>
     <plugin name="differential_drive_controller" filename="libgazebo_ros_diff_drive.so">

Commit message: 1/12

File: wheel_description/urdf/wheel.xacro (robot description, xacro)
@@ -103,9 +103,9 @@
   </joint>
   <joint type="continuous" name="right_wheel_hinge">
-    <origin xyz="-0.43 -0.26 0.28" rpy="-1.5707 0 0"/>
+    <origin xyz="-0.43 -0.26 0.28" rpy="1.5707 0 0"/>
     <!--origin xyz="0.1 -0.13 0" rpy="0 1.5707 1.5707"/-->
     <child link="right_wheel"/>
     <parent link="base_link"/>
-    <axis xyz="0 0 -1" rpy="0 0 0"/>
+    <axis xyz="0 0 1" rpy="0 0 0"/>
     <limit effort="10000" velocity="1000"/>
     <joint_properties damping="1.0" friction="1.0"/>
@@ -144,4 +144,10 @@
       </geometry>
     </collision>
+ <visual>
+      <origin xyz="0 0 0" rpy="0 0 0"/>
+      <geometry>
+        <mesh filename="package://rrbot_description/meshes/hokuyo.dae"/>
+      </geometry>
+    </visual>
     <inertial>
       <mass value="1e-5" />
@@ -152,5 +158,5 @@
  <joint name="imu_joint" type="fixed">
     <axis xyz="0 0 0" />
-    <origin xyz="0 0 0.75" rpy="0 0 0"/>
+    <origin xyz="0 0 0.63" rpy="0 0 0"/>
     <parent link="base_link"/>
     <child link="base_imu_link"/>

Commit message: global と　local wo を修正

File: wheel_description/urdf/wheel.xacro (robot description, xacro)
@@ -24,5 +24,7 @@
       </geometry>
     </visual>
-    <collision name='caster_collision'>
+</link>
+ <link name="caster_link">
+    <collision >
       <origin xyz="0 0 0.09" rpy=" 0 0 0"/>
       <geometry>
@@ -40,5 +42,5 @@
       </surface>
     </collision>
-    <visual name='caster_visual'>
+    <visual >
       <origin xyz="0 0 0.09" rpy=" 0 0 0"/>
       <geometry>
@@ -46,5 +48,21 @@
       </geometry>
     </visual>
-  </link>
+ <inertial>
+      <origin xyz="0 0 0"/>
+      <mass value="0.500"/>
+      <inertia ixx="0.00025" ixy="0" ixz="0" iyy="0.00025"  iyz="0" izz="0.00025"/>
+    </inertial>
+  </link>
+    <joint name="caster_joint" type="fixed">
+    <parent link="base_link"/>
+    <child link="caster_link"/>
+    <origin xyz="0 0 0"/>
+  </joint>
+<link name="base_footprint"/>
+  <joint name="base_link_joint" type="fixed">
+    <parent link="base_footprint"/>
+    <child link="base_link"/>
+    <origin xyz="0 0 0.100"/>
+  </joint>
   <link name="left_wheel">
     <!--origin xyz="0.1 0.13 0.1" rpy="0 1.5707 1.5707"/-->

Commit message: とりまうごく

File: wheel_description/urdf/wheel.xacro (robot description, xacro)
@@ -151,5 +151,5 @@
   <joint name="hokuyo_joint" type="fixed">
     <axis xyz="0 0 0" />
-    <origin xyz="0 0 0.63" rpy="0 0 0"/>
+    <origin xyz="0.1007 0 0.0558" rpy="0 0 0"/>
     <parent link="base_link"/>
     <child link="hokuyo_link"/>
@@ -176,5 +176,5 @@
  <joint name="imu_joint" type="fixed">
     <axis xyz="0 0 0" />
-    <origin xyz="0 0 0.63" rpy="0 0 0"/>
+    <origin xyz="0.1007 0 0.0558" rpy="0 0 0"/>
     <parent link="base_link"/>
     <child link="base_imu_link"/>

Commit message: last

File: wheel_description/urdf/wheel.xacro (robot description, xacro)
@@ -131,21 +131,4 @@
 <!-- Hokuyo Laser -->
   <link name="hokuyo_link">
-    <collision>
-      <origin xyz="0 0 0" rpy="0 0 0"/>
-      <geometry>
-        <box size="0.1 0.1 0.1"/>
-      </geometry>
-    </collision>
-    <visual>
-      <origin xyz="0 0 0" rpy="0 0 0"/>
-      <geometry>
-        <mesh filename="package://rrbot_description/meshes/hokuyo.dae"/>
-      </geometry>
-    </visual>
-    <inertial>
-      <mass value="1e-5" />
-      <origin xyz="0 0 0" rpy="0 0 0"/>
-      <inertia ixx="1e-6" ixy="0" ixz="0" iyy="1e-6" iyz="0" izz="1e-6" />
-    </inertial>
   </link>
   <joint name="hokuyo_joint" type="fixed">
@@ -156,21 +139,4 @@
   </joint>
  <link name="base_imu_link">
-    <collision>
-      <origin xyz="0 0 0" rpy="0 0 0"/>
-      <geometry>
-        <box size="0.1 0.1 0.1"/>
-      </geometry>
-    </collision>
- <visual>
-      <origin xyz="0 0 0" rpy="0 0 0"/>
-      <geometry>
-        <mesh filename="package://rrbot_description/meshes/hokuyo.dae"/>
-      </geometry>
-    </visual>
-    <inertial>
-      <mass value="1e-5" />
-      <origin xyz="0 0 0" rpy="0 0 0"/>
-      <inertia ixx="1e-6" ixy="0" ixz="0" iyy="1e-6" iyz="0" izz="1e-6" />
-    </inertial>
   </link>
  <joint name="imu_joint" type="fixed">
